File: MKS974_interface_board.kicad_sch (KiCad schematic)
At the start: 13 parts, among them J9 Barrel_Jack

Commit message: Add digikey listing to DB-9 and DB-15 ports
Parts:
- DB15-1, DB15-2, DB15-3, DB15-4: Listing (none) -> https://www.digikey.com/en/products/detail/amphenol-icc-fci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
Changed lines of the file:
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@@
 					(size 1.27 1.27)
 				)
+				(hide yes)
 			)
 		)
@@
 			)
 		)
-		(property "Description" ""
+		(property "Description" "https://www.digikey.com/en/products/detail/assmann-wsw-components/A-DS-09-A-KG-T4/21656068"
 			(at 25.4 77.47 0)
 			(effects
@@
 			)
 		)
+		(property "Listing" "https://www.digikey.com/en/products/detail/amphenol-icc-fci/ICD15S13E4GX00LF/1536501"
+			(at 33.02 186.69 90)
+			(effects
+				(font
+					(size 1.27 1.27)
+				)
+				(hide yes)
+			)
+		)
 		(pin "0"
 		)
@@
 			)
 		)
+		(property "Listing" "https://www.digikey.com/en/products/detail/amphenol-icc-fci/ICD15S13E4GX00LF/1536501"
+			(at 68.58 176.53 90)
+			(effects
+				(font
+					(size 1.27 1.27)
+				)
+				(hide yes)
+			)
+		)
 		(pin "0"
 		)
@@
 					(size 1.27 1.27)
 				)
+				(hide yes)
 			)
 		)
@@
 			)
 		)
-		(property "Description" ""
+		(property "Description" "https://www.digikey.com/en/products/detail/assmann-wsw-components/A-DS-09-A-KG-T4/21656068"
 			(at 60.96 66.04 0)
 			(effects
@@
 					(size 1.27 1.27)
 				)
+				(hide yes)
 			)
 		)
@@
 			)
 		)
-		(property "Description" ""
+		(property "Description" "https://www.digikey.com/en/products/detail/assmann-wsw-components/A-DS-09-A-KG-T4/21656068"
 			(at 95.25 55.88 0)
 			(effects
@@
 			)
 		)
+		(property "Listing" "https://www.digikey.com/en/products/detail/amphenol-icc-fci/ICD15S13E4GX00LF/1536501"
+			(at 139.7 156.21 90)
+			(effects
+				(font
+					(size 1.27 1.27)
+				)
+				(hide yes)
+			)
+		)
 		(pin "0"
 		)
@@
 			)
 		)
+		(property "Listing" "https://www.digikey.com/en/products/detail/amphenol-icc-fci/ICD15S13E4GX00LF/1536501"
+			(at 102.87 165.1 90)
+			(effects
+				(font
+					(size 1.27 1.27)
+				)
+				(hide yes)
+			)
+		)
 		(pin "0"
 		)
@@
 					(size 1.27 1.27)
 				)
+				(hide yes)
 			)
 		)
@@
 			)
 		)
-		(property "Description" ""
+		(property "Description" "https://www.digikey.com/en/products/detail/assmann-wsw-components/A-DS-09-A-KG-T4/21656068"
 			(at 132.08 46.99 0)
 			(effects
